Commit message: chore(robot): 구동 바퀴 지름 확정값 75mm 반영
부품표에서 75mm 로봇용 구동 바퀴로 확정됐다. 임시값 65mm 로 두면
주행 거리가 약 13% 짧게 계산돼 로봇이 지도에서 흘러간다.

1440 CPR 기준 1카운트당 0.164mm 이동, 이론 최고속도 0.479 m/s.
안전 상한은 0.25 m/s 를 유지한다. 화분을 이고 다니는 구조라 무게중심이
높고, 급가속하면 흔들려서 식물이 쏟아진다.

wheel_separation 은 섀시 조립 후 실측이 필요해 TODO 로 남긴다.

File: robot/src/potner_description/urdf/potner.urdf.xacro (robot description, xacro)
@@ -10,6 +10,6 @@
 <robot name="potner" xmlns:xacro="http://www.ros.org/wiki/xacro">
   <!-- ===== 실측 필요 (TODO) ===================================== -->
-  <xacro:property name="wheel_diameter"    value="0.065"/>  <!-- 구동 바퀴 지름 -->
-  <xacro:property name="wheel_width"       value="0.026"/>
+  <xacro:property name="wheel_diameter"    value="0.075"/>  <!-- 확정: 75mm 구동 바퀴 -->
+  <xacro:property name="wheel_width"       value="0.026"/>  <!-- TODO 실측 -->
   <xacro:property name="wheel_separation"  value="0.200"/>  <!-- 좌우 바퀴 중심 간 거리 -->
   <xacro:property name="body_diameter"     value="0.240"/>  <!-- 본체 외경 -->

Commit message: fix(base): 바퀴 지름을 실제 부품 값 60mm 로 정정
75mm 로 잘못 알고 있었습니다. 실제 구동 바퀴는 60mm 입니다.

퍼져 있던 여섯 곳을 한 번에 고쳤습니다 — kinematics 기본값, base_driver
declare_parameter, potner_params.yaml, URDF, 펌웨어 상수, 그리고 yaml 의
이론 최대속도 주석(122RPM x 60mm = 약 0.38 m/s).

이 값이 틀리면 두 가지가 동시에 어긋납니다.
- 오도메트리가 이동거리를 25% 과대보고 -> 지도가 실제보다 크게 그려짐
- PID 가 측정속도를 25% 과대평가 -> 실제 주행이 명령보다 20% 느림

한 곳만 고치는 실수는 test_config_consistency 와
test_firmware_constants 가 잡습니다. 이번에도 여섯 곳이 전부 같은
커밋에 있는 이유입니다.

286 tests passed, flake8 0

Refs: S15P11E104-349

File: robot/src/potner_description/urdf/potner.urdf.xacro (robot description, xacro)
@@ -10,5 +10,5 @@
 <robot name="potner" xmlns:xacro="http://www.ros.org/wiki/xacro">
   <!-- ===== 실측 필요 (TODO) ===================================== -->
-  <xacro:property name="wheel_diameter"    value="0.075"/>  <!-- 확정: 75mm 구동 바퀴 -->
+  <xacro:property name="wheel_diameter"    value="0.060"/>  <!-- 확정: 60mm 구동 바퀴 -->
   <xacro:property name="wheel_width"       value="0.026"/>  <!-- TODO 실측 -->
   <xacro:property name="wheel_separation"  value="0.200"/>  <!-- 좌우 바퀴 중심 간 거리 -->

Commit message: fix(base): 좌우 축간거리를 실측값 0.230m 으로 확정
자로 재니 바퀴 바깥면 사이가 25.5cm, 바퀴 두께가 2.5cm 였다. 중심 간
거리는 25.5 - 2.5 = 23.0cm 다. 그동안 쓰던 0.200 은 추측값이었고 실제보다
15% 작았다.

이 값은 두 곳에 동시에 쓰인다. cmd_vel 의 각속도를 좌우 바퀴 속도로 바꿀
때, 그리고 엔코더에서 회전각을 되계산할 때다. 두 곳이 같은 값을 쓰기
때문에 오차가 서로 상쇄되어 **오도메트리는 늘 명령한 만큼 돌았다고
보고하면서 몸만 덜 돈다.** 그래서 오도메트리로 닫아도 안 잡히고 실측
외에는 방법이 없었다.

실제로 어긋나던 것들:
  - 오도메트리 회전 보고가 실제보다 15% 큼 -> 지도가 회전할 때마다 뒤틀림
  - 수동 조작 22.5도 명령이 실제로는 19.6도
  - 도킹 후 180도 회전이 실제로는 156도

wheel_width 도 TODO 였는데 실측 2.5cm 로 채웠다 (RViz 표시용이라 기능
영향은 없다).

test_config_consistency 가 base_driver_node 의 declare_parameter 를
잡아냈다. 같은 값이 네 곳(yaml / declare_parameter / DriveConfig / URDF)에
흩어져 있어 하나를 빠뜨리기 쉬운데, 그러라고 있는 테스트다.

File: robot/src/potner_description/urdf/potner.urdf.xacro (robot description, xacro)
@@ -11,6 +11,6 @@
   <!-- ===== 실측 필요 (TODO) ===================================== -->
   <xacro:property name="wheel_diameter"    value="0.060"/>  <!-- 확정: 60mm 구동 바퀴 -->
-  <xacro:property name="wheel_width"       value="0.026"/>  <!-- TODO 실측 -->
-  <xacro:property name="wheel_separation"  value="0.200"/>  <!-- 좌우 바퀴 중심 간 거리 -->
+  <xacro:property name="wheel_width"       value="0.025"/>  <!-- 실측 -->
+  <xacro:property name="wheel_separation"  value="0.230"/>  <!-- 실측: 바깥면 25.5cm - 바퀴폭 2.5cm -->
   <xacro:property name="body_diameter"     value="0.240"/>  <!-- 본체 외경 -->
   <xacro:property name="body_height"       value="0.180"/>
